File: PCB/r2dtf dev board rev 1/r2dtf dev board rev 1.kicad_sch (KiCad schematic)
At the start: 11 parts, among them J1 Motor 1, J2 Motor 2, J5 Motor 1 Drive, J6 Motor 2 Drive, J7 External Power/VBAT In, J8 External Power/VBAT Out, SW1 External Power Switch

Commit message: Moved from library to my own motor functions, first working test of fast PWM
Other:
- note added: "Todo: Current Sense outputs have a 10k in series, but I am not sure I want to use them given possibility of exceeding VDD + 0.3 = 0.3 unpowered, 3.6 powered on Arduino nano Add test points everywhere Add decoupling caps Add larger power capacitor Solder a 0.1 µF ceramic capacitor across the terminals of your motors Max current: 12 A 5 minutes, 6 A indefinite Route your motor and power leads away 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"
- note removed: "Todo: Add test points everywhere Add decoupling caps Add larger power capacitor CHeck that there is no issue having this turned on and USB connected to arduino"

Commit message: Added Test Connectors, connected Arduino, rearranged
Parts:
- added C1, C2, C3, C4: C_Small_vert, symbol MyCapacitors:C_Small_vert
- added J10: M2 Test Enconder Connector, symbol MyConnectors:01x05_Connector
- added J11: Power Test Connector, symbol MyConnectors:01x04_Connector
- added J3: M1 Test Enconder Connector, symbol MyConnectors:01x04_Connector
- added J4: M2 Test Connector, symbol MyConnectors:01x05_Connector
- added J9: M1 Test Connector, symbol MyConnectors:01x05_Connector
- XA1: symbol PCM_arduino-library:Arduino_Nano_33_BLE_Sense_R2_Socket -> MyBoards:Arduino_Nano_33_BLE_Sense_R2_Socket
Connections:
- net +3V3: now also U1.3 (VDD-Input), C2.1, J11.3 (Pin_3); no longer U1. (VOUT-Rev_Prot_VBAT), U2.8 (OE)
- net +5V: now also XA1.VIN, C1.1, J11.2 (Pin_2)
- net GND: now also U1.1 (GND), C1.2, C2.2, J11.4 (Pin_4); no longer U1. (VOUT-Rev_Prot_VBAT)
- net at J2.1 (M2-Red-Power), J6.1 (Pin_1): now also C4.1
- net at J2.2 (M2-Black-Power), J6.2 (Pin_2): now also C4.2
- net M2-Enc_A-Yellow-5V: now reaches J2.5 (M2-Yellow-ENC_A), U2.4 (A3)
- net M2-Enc_A-Yellow-5V: now also J3.3 (Pin_3)
- net M2-Enc_B-White-5V: now reaches J2.6 (M2-White-ENC_B), U2.5 (A4)
- net M2-Enc_B-White-5V: now also J3.4 (Pin_4)
- net at J1.1 (M1-Red-Power), J5.1 (Pin_1): now also C3.1
- net at J1.2 (M1-Black-Power), J5.2 (Pin_2): now also C3.2
- net at SW1.1 (A): no longer J8.1 (Pin_1-VBAT)
- net VBAT: now reaches J7.1 (Pin_1-VBAT), SW1.2 (B)
- net VBAT: now also J11.1 (Pin_1)
- net at U3.2 (In_+_4.5-20V): now also U1.2 (VOUT-Rev_Protected_VBAT); no longer U1. (VOUT-Rev_Prot_VBAT)
- net M2-Enc_A-Yellow-3V3: now reaches XA1.A2 (A2/P0.30)
- net M2-Enc_A-Yellow-3V3: now also U2.11 (B3Y), J10.4 (Pin_4)
- net M2-Enc_B-White-3V3: now reaches XA1.A3 (A3/P0.29)
- net M2-Enc_B-White-3V3: now also U2.10 (B4Y), J10.5 (Pin_5)
- net M1-Enc_A-Yellow-3V3: now reaches XA1.A6 (A6/P0.28)
- net M1-Enc_A-Yellow-3V3: now also U2.13 (B1Y), J10.2 (Pin_2)
- net M1-Enc_B-White-3V3: now reaches XA1.A7 (A7/P0.03)
- net M1-Enc_B-White-3V3: now also U2.12 (B2Y), J10.3 (Pin_3)
- net M2_PWM: now reaches XA1.D10 (D10/P1.02/PWM)
- net M2_PWM: now also U1.12 (M2PWM), J4.4 (Pin_4)
- net M2_EN/DIAG: now reaches XA1.D12 (D12/P1.08/MISO)
- net M2_EN/DIAG: now also U1.9 (M2EN/DIAG), J4.1 (Pin_1)
- net M1_INA: now reaches XA1.D2 (D2/P1.11)
- net M1_INA: now also U1.5 (M1INA), J9.2 (Pin_2)
- net M1_INB: now reaches XA1.D4 (D4/P1.15)
- net M1_INB: now also U1.6 (M1INB), J9.3 (Pin_3)
- net TXU_OE: now reaches XA1.D5 (D5/P1.13/PWM)
- net TXU_OE: now also U2.8 (OE), J10.1 (Pin_1)
- net M1_EN/DIAG: now reaches XA1.D6 (D6/P1.14/PWM)
- net M1_EN/DIAG: now also U1.4 (M1EN/DIAG), J9.1 (Pin_1)
- net M2_INA: now reaches XA1.D7 (D7/P0.23)
- net M2_INA: now also U1.10 (M2INA), J4.2 (Pin_2)
- net M2_INB: now reaches XA1.D8 (D8/P0.21)
- net M2_INB: now also U1.11 (M2INB), J4.3 (Pin_3)
- net M1_PWM: now reaches XA1.D9 (D9/P0.27/PWM)
- net M1_PWM: now also U1.7 (M1PWM), J9.4 (Pin_4)
- net M1-Enc_A-Yellow-5V: now reaches J1.5 (M1-Yellow-ENC_A), U2.2 (A1)
- net M1-Enc_A-Yellow-5V: now also J3.1 (Pin_1)
- net M1-Enc_B-White-5V: now reaches J1.6 (M1-White-ENC_B), U2.3 (A2)
- net M1-Enc_B-White-5V: now also J3.2 (Pin_2)
- new net M1_CS: J9.5 (Pin_5), U1.8 (M1CS)
- new net M2_CS: J4.5 (Pin_5), U1.13 (M2CS)
Other:
- note added: "#define MOTOR_DRIVER_PIN_INA1 2 // M1INA Motor 1 direction input A #define MOTOR_DRIVER_PIN_INB1 4 // M1INB Motor 1 direction input B #define MOTOR_DRIVER_PIN_PWM1 9 // M1PWM Motor 1 speed input #define MOTOR_DRIVER_PIN_EN1DIAG1 6 // M1EN/DIAG Motor 1 enable input/fault output #define MOTOR_DRIVER_PIN_CS1 A0 // M1CS Motor 1 current sense output #define MOTOR_DRIVER_PIN_INA2 7 // M1INA Motor 2 dir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"
- note added: "Arduino board is powered from 5V Buck Board"
- note added: "Arduino board supplies 3V3 power"
- note added: "Battery switch on --> Arduino On/5 V power On: 1) OE of TXU0104 is disabled Motor INXA/B are both low so CS output is 0. 2) OE is enabled, passing Hall sensor signals through"
- note added: "NOTE: As opposed to other Arduino Nano boards, pins A4 and A5 have an internal pull up and default to be used as an I2C Bus so usage as analog inputs is not recommended. D11, 12, 13 are SPI"
- note added: "Todo: Test the use of analog pins as digital IO CHeck that there is no issue having this turned on and USB connected to arduino Add test points everywhere Add larger power capacitor Current Sense outputs have a 10k in series, but I am not sure I want to use them given possibility of exceeding VDD + 0.3 = 0.3 unpowered, 3.6 powered on Arduino nano Note that while the M1CS and M2CS voltages can pot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"
- note removed: "Todo: Current Sense outputs have a 10k in series, but I am not sure I want to use them given possibility of exceeding VDD + 0.3 = 0.3 unpowered, 3.6 powered on Arduino nano Add test points everywhere Add decoupling caps Add larger power capacitor Solder a 0.1 µF ceramic capacitor across the terminals of your motors Max current: 12 A 5 minutes, 6 A indefinite Route your motor and power leads away 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"
- moved on the sheet: J1, J2, J5, J6, J7, J8, SW1, U2
