File: PCB/r2dtf dev board rev 1/_autosave-r2dtf dev board rev 1.kicad_sch (KiCad schematic)
At the start: 23 parts, among them J1 BATT IN, J10 Power Test Connector, J11 M1 Test Connector, J12 M2 Test Connector, J13 5V Enconder Test Connector, J14 3V3 Enconder Test Connector, J2 Current Sense Jumper Out of b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, J3 Current Sense Jumper Into boa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, J4 Motor 1, J5 Motor 2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

Commit message: First pass at complete Rev 1. About to quote with JLCPCB
Connections:
- net M2 Red: now reaches C2.1, J5.1 (M2-Red-Power), J8.1 (Pin_1)
- net M2 Black: now reaches C2.2, J5.2 (M2-Black-Power), J8.2 (Pin_2)
- net M1 Red: now reaches C1.1, J4.1 (M1-Red-Power), J6.1 (Pin_1)
- net M1 Black: now reaches C1.2, J4.2 (M1-Black-Power), J6.2 (Pin_2)
- net BATT POST_SWITCH: now reaches J7.2 (Pin_2-VBAT), SW1.1 (A)
- net Post-Jumper CS2: now reaches J3.2 (Pin_2), XA1.A0 (A0/P0.04/DAC)
- net Post-Jumper CS1: now reaches J3.1 (Pin_1), XA1.A1 (A1/P0.05)
- net D11: now reaches J9.2 (Pin_2), XA1.D11 (D11/P1.01/MOSI)
- net D13: now reaches J9.3 (Pin_3), XA1.D13 (D13/P0.13/SCK/LED)
- net D3: now reaches J9.1 (Pin_1), XA1.D3 (D3/P1.12/PWM)
- net BATT GND: now reaches J1.2 (Pin_2-GND), J7.1 (Pin_1-GND)
Other:
- moved on the sheet: J2, J3
